File: Precharge Circuit/LV/LV.kicad_sch (KiCad schematic)
At the start: 9 parts

Commit message: Working on shutdown schematic
Parts:
- added D?: DIODE, symbol Simulation_SPICE:DIODE
- added K? (x2): ADW11, Relay_THT:Relay_1P1T_NO_10x24x18.8mm_Panasonic_ADW11xxxxW_THT, symbol Relay:ADW11
- added R?: 500, symbol Device:R_US
- added U: Right Shutdown, Package_DIP:DIP-8_W7.62mm, symbol Analog_Switch:ADG417BN
- added U: Left Shutdown, Package_DIP:DIP-8_W7.62mm, symbol Analog_Switch:ADG417BN
- added U: BOTS, Package_DIP:DIP-8_W7.62mm, symbol Analog_Switch:ADG417BN
- added U: Cockpit Shutdown, Package_DIP:DIP-8_W7.62mm, symbol Analog_Switch:ADG417BN
- added U: TS Master Switch, Package_DIP:DIP-8_W7.62mm, symbol Analog_Switch:ADG417BN
- added U?: HVD Interlock, Package_DIP:DIP-8_W7.62mm, symbol Analog_Switch:ADG417BN
- added U?: ADG417BN, Package_DIP:DIP-8_W7.62mm, symbol Analog_Switch:ADG417BN
- added U?: Intertia Switch, Package_DIP:DIP-8_W7.62mm, symbol Analog_Switch:ADG417BN
Connections:
- net GND: now also Q?.3 (E), K?.1
- net IMD Out: now reaches K?.6, R.2, R.2
- net ECU +5: now reaches R.1
- net ECU +5: now also R?.2
- net at K?.3: now also K?.5
- net at K?.5: now also K?.3, U?.8
- net at K?.3: now also U.8
- net at Q?.1 (B): now also D?.2 (K)
- new net: U.1, U?.8
- new net: U.1, U.8 (x3)
- new net: K?.5, U?.1
- new net: D?.1 (A), R?.1
- new net: K?.5, K?.6, U.1, U?.1
- new net: K?.3, U?.8
- new net 1out: K?.1
- new net 2out: K?.6
Other:
- added sheet ECU Pinout (untitled.kicad_sch)
- title: (none) -> RM27 Shutdown Circuit
- moved on the sheet: D?, K?, Q?, R
