File: LV/LV.kicad_sch (KiCad schematic)
At the start: 21 parts

Commit message: Updates to LV Schematic
Parts:
- added D1: LED, symbol Device:LED
- added U1: HV+ Interlock, Package_DIP:DIP-8_W7.62mm, symbol Analog_Switch:ADG417BN
- added U2: HV- Interlock, Package_DIP:DIP-8_W7.62mm, symbol Analog_Switch:ADG417BN
- D?: value ${SIM.PARAMS} -> IMD LED
- D?: value ${SIM.PARAMS} -> AMS LED (moved???)
Connections:
- net GND: now also D1.1 (K)
- net 12V+: now reaches U?.1
- net Inverter Power: now reaches U.8
- net Inverter Power: now also U1.1
- new net: U1.8, U2.1
- new net Shutdown out: D1.2 (A), U2.8
