File: Precharge Circuit/Precharge/Precharge.kicad_sch (KiCad schematic)
At the start: 2 parts

Commit message: Update
Parts:
- removed A1: Arduino_Nano_ESP32_Socket, PCM_arduino-library:Arduino_Nano_ESP32_Socket, symbol PCM_arduino-library:Arduino_Nano_ESP32_Socket
- removed K1: ~, symbol PrechargeRelays:PreDisRelay
- added A1: Arduino_Nano_33_IoT_Socket, PCM_arduino-library:Arduino_Nano_33_IoT_Socket, symbol PCM_arduino-library:Arduino_Nano_33_IoT_Socket
- added C1, C11, C12: C324C106K3R5TA, 10uF Cap:CAP_C324C_MR_X7R_KEM, symbol 10uF Cap:C324C106K3R5TA
- added C10, C6, C7, C9: K331K15X7RF5TL2, 330pFCap:CAP_K-SERIES_15-L2_VIS, symbol 330pF Cap:K331K15X7RF5TL2
- added C2, C3, C4, C5, C8: K104K10X7RF5UH5, 1uFCap:K104K10X7RF5UH5_VIS, symbol 1u Cap:K104K10X7RF5UH5
- added CR1, CR2: B240A-13-F, PreChargeParts:SMA_DIO-L, symbol RelayFlyback:B240A-13-F
- added J1, J2: 430450428, MolexVertical:CONN_SD-43045-010_04_MOL, symbol 4PinMictrofit:430450428
- added J4: 436500228, MolexVertical:CONN_SD-43650-010_02_MOL, symbol 2PinMicro-FitV:436500228
- added MOSFET1, MOSFET2: DMN3404L-7, PreChargeParts:SOT23_DIO-L, symbol RelayFET:DMN3404L-7
- added PS1: R-78E5.0-0.5, 12-5V Converter:CONV_R-78E5.0-0.5, symbol R-78E5.0-0.5:R-78E5.0-0.5
- added R1, R13, R14, R15, R16, R17, R2, R3, R4, R5: 200k, Resistor_THT:R_Axial_DIN0207_L6.3mm_D2.5mm_P10.16mm_Horizontal, symbol Device:R_US
- added R10, R21, R22, R9: 1k, Resistor_THT:R_Axial_DIN0207_L6.3mm_D2.5mm_P10.16mm_Horizontal, symbol Device:R_US
- added R11, R12, R23, R24: 2.5k, Resistor_THT:R_Axial_DIN0207_L6.3mm_D2.5mm_P10.16mm_Horizontal, symbol Device:R_US
- added R18, R26, R28, R6: 10k, Resistor_THT:R_Axial_DIN0207_L6.3mm_D2.5mm_P10.16mm_Horizontal, symbol Device:R_US
- added R25, R27: 200, Resistor_THT:R_Axial_DIN0207_L6.3mm_D2.5mm_P10.16mm_Horizontal, symbol Device:R_US
- added U1: TEA 1-0505E, PreChargeParts:TEA 1E_TRP, symbol Isolating DC-DC Converter:TEA_1-0505E
- added U2, U3: AMC1351DWVR, AMC 1351:SOIC8_DWV_TEX, symbol AMC 1351:AMC1351DWVR
- added U6: OP284EPZ, OP284:N_8_ADI, symbol OP284:OP284EPZ
Connections:
- new net: R17.2, R18.2, U3.2 (IN)
- new net: J2.3, R13.1
- new net: J2.4, R1.1
- new net: C10.1, R21.2, R23.2, U6.5 (+INB)
- new net: R1.2, R2.1
- new net: R2.2, R3.1
- new net: R4.2, R5.1
- new net: R5.2, R6.2, U2.2 (IN)
- new net: J4.2, PS1.1 (+VIN)
- new net: R22.1, U3.6 (OUTN)
- new net: C9.1, R22.2, R24.2, U6.6 (-INB)
- new net: R10.1, U2.7 (OUTP)
- new net: C6.1, R10.2, R12.2, U6.3 (+INA)
- new net: R16.2, R17.1
- new net: R3.2, R4.1
- new net: R9.1, U2.6 (OUTN)
- new net: C7.1, R11.2, R9.2, U6.2 (-INA)
- new net: MOSFET1.1 (G), R25.2, R26.1
- new net: CR1.2, J1.2, MOSFET1.3 (D)
- new net: R13.2, R14.1
- new net: R14.2, R15.1
- new net: A1.A2, C9.2, R24.1, U6.7 (OUTB)
- new net: A1.A7, C7.2, R11.1, U6.1 (OUTA)
- new net: R21.1, U3.7 (OUTP)
- new net: R15.2, R16.1
- new net: A1.D2, R25.1
- new net: A1.D3, R27.1
- new net: MOSFET2.1 (G), R27.2, R28.1
- new net: CR2.2, J1.3, MOSFET2.3 (D)
- new net +5: A1.VIN, C1.1, C12.1, C3.1, C5.1, C8.1, PS1.3 (+VOUT), U1.1 (+VIN(VCC)), U2.8 (VDD2), U3.8 (VDD2), U6.8 (V+)
- new net GND: A1.GND1 (GND), A1.GND2 (GND), C1.2, C10.2, C12.2, C3.2, C5.2, C6.2, C8.2, J1.4, J4.1, MOSFET1.2 (S), MOSFET2.2 (S), PS1.2 (GND), R12.1, R23.1, R26.2, R28.2, U1.2 (-VIN(GND)), U2.5 (GND2), U3.5 (GND2), U6.4 (V-)
- new net HV+5: C11.1, C2.1, C4.1, U1.6 (+VOUT), U2.1 (VDD1), U3.1 (VDD1)
- new net HVGND: C11.2, C2.2, C4.2, J2.1, J2.2, R18.1, R6.1, U1.4 (-VOUT), U2.3 (GND1), U2.4 (GND1), U3.3 (GND1), U3.4 (GND1)
- new net ShutdownIn: CR1.1, CR2.1, J1.1
Other:
- note added: "HV Sense Inputs (Battery Voltage and Inverter Voltage)"
- note added: "Precharge Schematic"
- note added: "Relay Driver Outputs (Positive AIR and Precharge Relay)"
- company: (none) -> Blake Hopper
- title: (none) -> RM28 Precharge PCB
